Commit message: feature/rviz-core : update robot.urdf.xacro and readme.md

File: xacro/robot.urdf.xacro (robot description, xacro)
@@ -42,5 +42,5 @@
   <link name="base_plate">
     <visual>
-      <origin xyz="-0.39 -0.39 -0.56" rpy="0 0 0"/>
+      <origin xyz="0 0 0" rpy="0 0 0"/>
       <geometry>
         <mesh filename="package://industrial_arm_description/meshes/base_plate.stl" scale="${mesh_scale}"/>
@@ -56,5 +56,5 @@
     <parent link="base_plate"/>
     <child link="forward_drive_arm"/>
-    <origin xyz="0 0 0.035" rpy="0 0 0"/>
+    <origin xyz="0 0 0.03" rpy="0 -${PI/2} ${PI/2}"/>
     <axis xyz="0 1 0"/>
     <limit lower="-${PI/2}" upper="${PI/2}" effort="${joint_effort}" velocity="${joint_velocity}"/>
@@ -62,5 +62,5 @@
   <link name="forward_drive_arm">
     <visual>
-      <origin xyz="0.19 0.06 -0.08" rpy="0 -${PI/2} ${PI/2}"/>
+      <origin xyz="0 0 0" rpy="0 0 0"/>
       <geometry>
         <mesh filename="package://industrial_arm_description/meshes/forward_drive_arm.stl" scale="${mesh_scale}"/>
@@ -76,5 +76,5 @@
     <parent link="forward_drive_arm"/>
     <child link="horizontal_arm"/>
-    <origin xyz="0 0 0.08" rpy="0 0 0"/>
+    <origin xyz="0 0 0.08" rpy="${PI/2} 0 ${PI/2}"/>
     <axis xyz="0 1 0"/>
     <limit lower="-${PI/2}" upper="${PI/2}" effort="${joint_effort}" velocity="${joint_velocity}"/>
@@ -82,5 +82,5 @@
   <link name="horizontal_arm">
     <visual>
-      <origin xyz="0.03 -0.4 -0.06" rpy="${PI/2} 0 ${PI/2}"/>
+      <origin xyz="0 0 0" rpy="0 0 0"/>
       <geometry>
         <mesh filename="package://industrial_arm_description/meshes/horizontal_arm.stl" scale="${mesh_scale}"/>
@@ -96,5 +96,5 @@
     <parent link="horizontal_arm"/>
     <child link="claw_support"/>
-    <origin xyz="0.082 0 0" rpy="0 0 0"/>
+    <origin xyz="0.082 0 0" rpy="0 0 ${PI/2}"/>
     <axis xyz="0 0 1"/>
     <limit lower="-${PI/2}" upper="${PI/2}" effort="${joint_effort}" velocity="${joint_velocity}"/>
@@ -102,5 +102,5 @@
   <link name="claw_support">
     <visual>
-      <origin rpy="0 0 ${PI/2}" xyz="0 -0.05 -0.15"/>
+      <origin xyz="0 0 0" rpy="0 0 0"/>
       <geometry>
         <mesh filename="package://industrial_arm_description/meshes/claw_support.stl" scale="${mesh_scale}"/>
@@ -116,5 +116,5 @@
     <parent link="claw_support"/>
     <child link="gripper_right"/>
-    <origin xyz="0.01 -0.004 -0.01" rpy="0 0 -${PI/2}"/>
+    <origin xyz="0 -0.01 0" rpy="0 0 -${PI/2}"/>
     <axis xyz="1 0 0"/>
     <limit lower="0.0" upper="0.022" effort="10.0" velocity="0.5"/>
@@ -122,5 +122,5 @@
   <link name="gripper_right">
     <visual>
-      <origin xyz="-0.1 0.5 -0.1" rpy="0 0 -${PI/2}"/>
+      <origin xyz="0 0 0" rpy="0 0 0"/>
       <geometry>
         <mesh filename="package://industrial_arm_description/meshes/gripper_right.stl" scale="${mesh_scale}"/>
@@ -136,5 +136,5 @@
     <parent link="claw_support"/>
     <child link="gripper_left"/>
-    <origin xyz="0.01 0.004 -0.01" rpy="0 0 -${PI/2}"/>
+    <origin xyz="0 0.01 0" rpy="0 0 -${PI/2}"/>
     <axis xyz="1 0 0"/>
     <limit lower="0.0" upper="0.022" effort="10.0" velocity="0.5"/>
@@ -143,5 +143,5 @@
   <link name="gripper_left">
     <visual>
-      <origin xyz="-0.04 0.5 -0.1" rpy="0 0 -${PI/2}"/>
+      <origin xyz="0 0 0" rpy="0 0 0"/>
       <geometry>
         <mesh filename="package://industrial_arm_description/meshes/gripper_left.stl" scale="${mesh_scale}"/>
